Commit message: rename sai2 to sai

File: config_folder/robot_files/iiwa7_plate.urdf (robot description, URDF)
Before this commit: robot kuka_iiwa, 9 links, 8 joints
Links:
- link base_link: geometry visual mesh filename=${SAI_MODEL_URDF_FOLDER}/iiwa7/meshes/base.obj scale=1 1 1
- link link0: geometry visual mesh filename=${SAI_MODEL_URDF_FOLDER}/iiwa7/meshes/link0.obj scale=1 1 1
- link link1: geometry visual mesh filename=${SAI_MODEL_URDF_FOLDER}/iiwa7/meshes/link1.obj scale=1 1 1
- link link2: geometry visual mesh filename=${SAI_MODEL_URDF_FOLDER}/iiwa7/meshes/link2.obj scale=1 1 1
- link link3: geometry visual mesh filename=${SAI_MODEL_URDF_FOLDER}/iiwa7/meshes/link3.obj scale=1 1 1
- link link4: geometry visual mesh filename=${SAI_MODEL_URDF_FOLDER}/iiwa7/meshes/link4.obj scale=1 1 1
- link link5: geometry visual mesh filename=${SAI_MODEL_URDF_FOLDER}/iiwa7/meshes/link5.obj scale=1 1 1
- link link6: geometry visual mesh filename=${SAI_MODEL_URDF_FOLDER}/iiwa7/meshes/link6.obj scale=1 1 1

File: config_folder/robot_files/panda_arm_peg.urdf (robot description, URDF)
Before this commit: robot panda, 9 links, 8 joints
Links:
- link link0: geometry visual mesh filename=${SAI_MODEL_URDF_FOLDER}/panda/meshes/visual/link0.obj
- link link1: geometry visual mesh filename=${SAI_MODEL_URDF_FOLDER}/panda/meshes/visual/link1.obj
- link link2: geometry visual mesh filename=${SAI_MODEL_URDF_FOLDER}/panda/meshes/visual/link2.obj
- link link3: geometry visual mesh filename=${SAI_MODEL_URDF_FOLDER}/panda/meshes/visual/link3.obj
- link link4: geometry visual mesh filename=${SAI_MODEL_URDF_FOLDER}/panda/meshes/visual/link4.obj
- link link5: geometry visual mesh filename=${SAI_MODEL_URDF_FOLDER}/panda/meshes/visual/link5.obj
- link link6: geometry visual mesh filename=${SAI_MODEL_URDF_FOLDER}/panda/meshes/visual/link6.obj
- link link7: geometry visual mesh filename=${SAI_MODEL_URDF_FOLDER}/panda/meshes/visual/link7.obj
