Commit message: Updated Reinforcement learning notebook:
Added Q learning models and notebook for demo

File: config_folder/robot_files/mobile_base.urdf (robot description, URDF)
Before this commit: robot panda, 13 links, 12 joints
Links:
- link end-effector: geometry visual cylinder length=0.08 radius=0.015
