Commit message: intermediate test

File: tutorials/tuto_config_folder/robot_files/pendulum.urdf (robot description, URDF)
Before this commit: robot pendulum, 2 links, 1 joints
Links:
- link link1: geometry visual cylinder length=1 radius=0.07; visual sphere radius=0.1

Commit message: more steps in tuto 1

File: tutorials/tuto_config_folder/robot_files/pendulum.urdf (robot description, URDF)
Before this commit: robot pendulum, 2 links, 1 joints
Links:
- added link link2, mass 1.0; visual cylinder length=1 radius=0.07; visual sphere radius=0.1
Joints:
- removed joint j0
- added joint j1: type revolute, parent base_link, child link1, origin xyz=0 0 0, axis 1 0 0, limit lower=-2.967 upper=2.967 effort=176 velocity=1.7104
- added joint j2: type revolute, parent link1, child link2, origin xyz=0 0 -1, axis 1 0 0, limit lower=-2.967 upper=2.967 effort=176 velocity=1.7104

Commit message: more tuto 1 steps

File: tutorials/tuto_config_folder/robot_files/pendulum.urdf (robot description, URDF)
Before this commit: robot pendulum, 3 links, 2 joints
Joints:
- joint j1: limit lower=-2.967 upper=2.967 effort=176 velocity=1.7104 -> lower=-0.967 upper=0.967 effort=176 velocity=1.7104
- joint j2: limit lower=-2.967 upper=2.967 effort=176 velocity=1.7104 -> lower=-0.967 upper=0.967 effort=176 velocity=1.7104

Commit message: finish tuto 1

File: tutorials/tuto_config_folder/robot_files/pendulum.urdf (robot description, URDF)
Before this commit: robot pendulum, 3 links, 2 joints
Links:
- removed link link2
- link link1: geometry visual cylinder length=1 radius=0.07
Joints:
- removed joint j2
- joint j1: limit lower=-0.967 upper=0.967 effort=176 velocity=1.7104 -> lower=-2.967 upper=2.967 effort=176 velocity=1.7104
